Commit message: Cleaned workspace and kept current files

File: urdf/arm.urdf (robot description, URDF)
Before this commit: robot rover_arm, 15 links, 14 joints
Links:
- added link world
Joints:
- removed joint joint_1_base_yaw
- removed joint joint_2_shoulder_pitch
- removed joint joint_3_elbow_pitch
- removed joint joint_4_wrist_roll
- removed joint joint_5_wrist_pitch
- added joint j0_base_yaw: type revolute, parent base_link, child robolink_1_disc, origin xyz=0 0 0.05 rpy=0 0 0, axis 0 0 1, limit lower=-3.14159 upper=3.14159 effort=30 velocity=1.0
- added joint j1_shoulder_pitch: type revolute, parent vertical_mast, child robolink_2_disc, origin xyz=0 0 0.060 rpy=0 0 0, axis 0 1 0, limit lower=-1.57 upper=2.60 effort=60 velocity=0.8
- added joint j2_elbow_pitch: type revolute, parent upper_arm, child robolink_3_disc, origin xyz=0.425 0 0 rpy=0 0 0, axis 0 1 0, limit lower=-2.35 upper=2.35 effort=40 velocity=1.0
- added joint j3_wrist_pitch: type revolute, parent forearm, child robolink_4_disc, origin xyz=0.470 0 0 rpy=0 0 0, axis 0 1 0, limit lower=-1.5708 upper=1.5708 effort=15 velocity=1.5
- added joint j4_wrist_roll: type revolute, parent robolink_4_disc, child wrist_bracket, origin xyz=0.018 0 0 rpy=0 0 0, axis 1 0 0, limit lower=-3.14159 upper=3.14159 effort=10 velocity=1.5
- added joint world_to_rover_deck: type fixed, parent world, child base_link, origin xyz=0 0 0.355 rpy=0 0 0
